Commit message: replace with old xacro

File: robot_description/urdf/robot.xacro (robot description, xacro)
@@ -6,5 +6,5 @@
 <link name="base_link">
   <inertial>
-    <origin xyz="0.03180031010101302 4.6312625487061606e-05 0.27555741033921555" rpy="0 0 0"/>
+    <origin xyz="0.03180031010101345 4.6312625487061606e-05 0.10698441033921668" rpy="0 0 0"/>
     <mass value="17.719416949374274"/>
     <inertia ixx="0.704305" iyy="1.004356" izz="1.471877" ixy="0.000745" iyz="0.000142" ixz="-0.000419"/>
@@ -26,10 +26,10 @@
 <link name="right_big_pivot_1">
   <inertial>
-    <origin xyz="-0.05850399376662565 -0.10854732888759794 -0.07469415008342872" rpy="0 0 0"/>
+    <origin xyz="-0.058503993766625226 -0.108547328887598 -0.07469415008342761" rpy="0 0 0"/>
     <mass value="2.2415377387384887"/>
     <inertia ixx="0.033507" iyy="0.078447" izz="0.086535" ixy="-2e-05" iyz="1e-06" ixz="-0.014743"/>
   </inertial>
   <visual>
-    <origin xyz="-0.032254 0.238359 -0.327323" rpy="0 0 0"/>
+    <origin xyz="-0.032254 0.238359 -0.15875" rpy="0 0 0"/>
     <geometry>
       <mesh filename="package://robot_description/meshes/right_big_pivot_1.stl" scale="0.001 0.001 0.001"/>
@@ -38,5 +38,5 @@
   </visual>
   <collision>
-    <origin xyz="-0.032254 0.238359 -0.327323" rpy="0 0 0"/>
+    <origin xyz="-0.032254 0.238359 -0.15875" rpy="0 0 0"/>
     <geometry>
       <mesh filename="package://robot_description/meshes/right_big_pivot_1.stl" scale="0.001 0.001 0.001"/>
@@ -46,10 +46,10 @@
 <link name="left_big_pivot_1">
   <inertial>
-    <origin xyz="-0.05850399376799906 0.10862267111240001 -0.07469415008342606" rpy="0 0 0"/>
+    <origin xyz="-0.05850399376799863 0.10862267111240007 -0.07469415008342495" rpy="0 0 0"/>
     <mass value="2.2415377387384736"/>
     <inertia ixx="0.033507" iyy="0.078447" izz="0.086535" ixy="-2e-05" iyz="1e-06" ixz="-0.014743"/>
   </inertial>
   <visual>
-    <origin xyz="-0.032254 -0.2386 -0.327323" rpy="0 0 0"/>
+    <origin xyz="-0.032254 -0.2386 -0.15875" rpy="0 0 0"/>
     <geometry>
       <mesh filename="package://robot_description/meshes/left_big_pivot_1.stl" scale="0.001 0.001 0.001"/>
@@ -58,5 +58,5 @@
   </visual>
   <collision>
-    <origin xyz="-0.032254 -0.2386 -0.327323" rpy="0 0 0"/>
+    <origin xyz="-0.032254 -0.2386 -0.15875" rpy="0 0 0"/>
     <geometry>
       <mesh filename="package://robot_description/meshes/left_big_pivot_1.stl" scale="0.001 0.001 0.001"/>
@@ -66,10 +66,10 @@
 <link name="right_little_pivot_1">
   <inertial>
-    <origin xyz="-0.00022083740446587896 -0.10783247162867271 -0.03446395454594753" rpy="0 0 0"/>
+    <origin xyz="-0.00022083740446540712 -0.10783247162867271 -0.034463954545946425" rpy="0 0 0"/>
     <mass value="1.158287566383538"/>
     <inertia ixx="0.010707" iyy="0.01462" izz="0.023908" ixy="-1e-06" iyz="-0.000121" ixz="8.5e-05"/>
   </inertial>
   <visual>
-    <origin xyz="-0.207006 -0.452595 -0.168573" rpy="0 0 0"/>
+    <origin xyz="-0.207006 -0.452595 -0.0" rpy="0 0 0"/>
     <geometry>
       <mesh filename="package://robot_description/meshes/right_little_pivot_1.stl" scale="0.001 0.001 0.001"/>
@@ -78,5 +78,5 @@
   </visual>
   <collision>
-    <origin xyz="-0.207006 -0.452595 -0.168573" rpy="0 0 0"/>
+    <origin xyz="-0.207006 -0.452595 -0.0" rpy="0 0 0"/>
     <geometry>
       <mesh filename="package://robot_description/meshes/right_little_pivot_1.stl" scale="0.001 0.001 0.001"/>
@@ -86,10 +86,10 @@
 <link name="left_little_pivot_1">
   <inertial>
-    <origin xyz="-0.00022083740307932143 0.10298752837132685 -0.03446395454594536" rpy="0 0 0"/>
+    <origin xyz="-0.00022083740307884958 0.10298752837132691 -0.03446395454594424" rpy="0 0 0"/>
     <mass value="1.158287566383538"/>
     <inertia ixx="0.010707" iyy="0.01462" izz="0.023908" ixy="-1e-06" iyz="-0.000121" ixz="8.5e-05"/>
   </inertial>
   <visual>
-    <origin xyz="-0.207006 0.452481 -0.168573" rpy="0 0 0"/>
+    <origin xyz="-0.207006 0.452481 -0.0" rpy="0 0 0"/>
     <geometry>
       <mesh filename="package://robot_description/meshes/left_little_pivot_1.stl" scale="0.001 0.001 0.001"/>
@@ -98,5 +98,5 @@
   </visual>
   <collision>
-    <origin xyz="-0.207006 0.452481 -0.168573" rpy="0 0 0"/>
+    <origin xyz="-0.207006 0.452481 -0.0" rpy="0 0 0"/>
     <geometry>
       <mesh filename="package://robot_description/meshes/left_little_pivot_1.stl" scale="0.001 0.001 0.001"/>
@@ -106,10 +106,10 @@
 <link name="wheel_1">
   <inertial>
-    <origin xyz="-2.3343628063887678e-07 -0.08910709857161447 4.492056740468264e-09" rpy="0 0 0"/>
-    <mass value="11.601933377005569"/>
-    <inertia ixx="0.066678" iyy="0.074767" izz="0.066678" ixy="0.0" iyz="0.0" ixz="-0.0"/>
-  </inertial>
-  <visual>
-    <origin xyz="0.31725 -0.452595 -0.073323" rpy="0 0 0"/>
+    <origin xyz="-2.3343628013927642e-07 -0.08910709857161442 4.492057850691289e-09" rpy="0 0 0"/>
+    <mass value="11.601933377005569"/>
+    <inertia ixx="0.066678" iyy="0.074767" izz="0.066678" ixy="0.0" iyz="0.0" ixz="-0.0"/>
+  </inertial>
+  <visual>
+    <origin xyz="0.31725 -0.452595 0.09525" rpy="0 0 0"/>
     <geometry>
       <mesh filename="package://robot_description/meshes/wheel_1.stl" scale="0.001 0.001 0.001"/>
@@ -118,5 +118,5 @@
   </visual>
   <collision>
-    <origin xyz="0.31725 -0.452595 -0.073323" rpy="0 0 0"/>
+    <origin xyz="0.31725 -0.452595 0.09525" rpy="0 0 0"/>
     <geometry>
       <mesh filename="package://robot_description/meshes/wheel_1.stl" scale="0.001 0.001 0.001"/>
@@ -126,10 +126,10 @@
 <link name="wheel_2">
   <inertial>
-    <origin xyz="-0.38150331945529364 -0.039295098571614784 -0.5403554023304846" rpy="0 0 0"/>
-    <mass value="11.601933377005569"/>
-    <inertia ixx="0.066678" iyy="0.074767" izz="0.066678" ixy="0.0" iyz="0.0" ixz="-0.0"/>
-  </inertial>
-  <visual>
-    <origin xyz="-0.410225 -0.402783 -0.633868" rpy="0 0 0"/>
+    <origin xyz="-3.1945529308657905e-07 -0.0891070985716147 -4.0233048348436995e-07" rpy="0 0 0"/>
+    <mass value="11.601933377005569"/>
+    <inertia ixx="0.066678" iyy="0.074767" izz="0.066678" ixy="0.0" iyz="0.0" ixz="-0.0"/>
+  </inertial>
+  <visual>
+    <origin xyz="-0.028722 -0.452595 0.07506" rpy="0 0 0"/>
     <geometry>
       <mesh filename="package://robot_description/meshes/wheel_2.stl" scale="0.001 0.001 0.001"/>
@@ -138,5 +138,5 @@
   </visual>
   <collision>
-    <origin xyz="-0.410225 -0.402783 -0.633868" rpy="0 0 0"/>
+    <origin xyz="-0.028722 -0.452595 0.07506" rpy="0 0 0"/>
     <geometry>
       <mesh filename="package://robot_description/meshes/wheel_2.stl" scale="0.001 0.001 0.001"/>
@@ -146,10 +146,10 @@
 <link name="wheel_3">
   <inertial>
-    <origin xyz="-0.3815036036551207 -0.04157109857161467 -0.5426314668854645" rpy="0 0 0"/>
-    <mass value="11.601933377005569"/>
-    <inertia ixx="0.066678" iyy="0.074767" izz="0.066678" ixy="0.0" iyz="0.0" ixz="-0.0"/>
-  </inertial>
-  <visual>
-    <origin xyz="-0.765818 -0.405059 -0.633868" rpy="0 0 0"/>
+    <origin xyz="3.963448797494884e-07 -0.08910709857161458 -4.6688546337381176e-07" rpy="0 0 0"/>
+    <mass value="11.601933377005569"/>
+    <inertia ixx="0.066678" iyy="0.074767" izz="0.066678" ixy="0.0" iyz="0.0" ixz="-0.0"/>
+  </inertial>
+  <visual>
+    <origin xyz="-0.384314 -0.452595 0.077336" rpy="0 0 0"/>
     <geometry>
       <mesh filename="package://robot_description/meshes/wheel_3.stl" scale="0.001 0.001 0.001"/>
@@ -158,5 +158,5 @@
   </visual>
   <collision>
-    <origin xyz="-0.765818 -0.405059 -0.633868" rpy="0 0 0"/>
+    <origin xyz="-0.384314 -0.452595 0.077336" rpy="0 0 0"/>
     <geometry>
       <mesh filename="package://robot_description/meshes/wheel_3.stl" scale="0.001 0.001 0.001"/>
@@ -166,10 +166,10 @@
 <link name="wheel_4">
   <inertial>
-    <origin xyz="-0.3591342334348961 0.11899490142838393 -0.06408999550794109" rpy="0 0 0"/>
-    <mass value="11.601933377005569"/>
-    <inertia ixx="0.066678" iyy="0.074767" izz="0.066678" ixy="0.0" iyz="0.0" ixz="-0.0"/>
-  </inertial>
-  <visual>
-    <origin xyz="-0.041884 0.449636 -0.137413" rpy="0 0 0"/>
+    <origin xyz="-2.3343489585769817e-07 -0.08910709857161611 4.4920600433817626e-09" rpy="0 0 0"/>
+    <mass value="11.601933377005569"/>
+    <inertia ixx="0.066678" iyy="0.074767" izz="0.066678" ixy="0.0" iyz="0.0" ixz="-0.0"/>
+  </inertial>
+  <visual>
+    <origin xyz="0.31725 0.241534 0.09525" rpy="0 0 0"/>
     <geometry>
       <mesh filename="package://robot_description/meshes/wheel_4.stl" scale="0.001 0.001 0.001"/>
@@ -178,5 +178,5 @@
   </visual>
   <collision>
-    <origin xyz="-0.041884 0.449636 -0.137413" rpy="0 0 0"/>
+    <origin xyz="0.31725 0.241534 0.09525" rpy="0 0 0"/>
     <geometry>
       <mesh filename="package://robot_description/meshes/wheel_4.stl" scale="0.001 0.001 0.001"/>
@@ -186,10 +186,10 @@
 <link name="wheel_5">
   <inertial>
-    <origin xyz="-0.38150331945390625 -0.07190017040328195 0.36472058868693286" rpy="0 0 0"/>
+    <origin xyz="-3.1945390568249854e-07 0.0891078295967182 -4.1131306602326667e-07" rpy="0 0 0"/>
     <mass value="11.601933377005569"/>
     <inertia ixx="0.066678" iyy="0.074767" izz="0.066678" ixy="-0.0" iyz="0.0" ixz="0.0"/>
   </inertial>
   <visual>
-    <origin xyz="-0.410225 0.291473 0.271208" rpy="0 0 0"/>
+    <origin xyz="-0.028722 0.452481 0.07506" rpy="0 0 0"/>
     <geometry>
       <mesh filename="package://robot_description/meshes/wheel_5.stl" scale="0.001 0.001 0.001"/>
@@ -198,5 +198,5 @@
   </visual>
   <collision>
-    <origin xyz="-0.410225 0.291473 0.271208" rpy="0 0 0"/>
+    <origin xyz="-0.028722 0.452481 0.07506" rpy="0 0 0"/>
     <geometry>
       <mesh filename="package://robot_description/meshes/wheel_5.stl" scale="0.001 0.001 0.001"/>
@@ -206,10 +206,10 @@
 <link name="wheel_6">
   <inertial>
-    <origin xyz="-0.3815036036537347 -0.07417617040328273 0.3624445241319522" rpy="0 0 0"/>
+    <origin xyz="3.9634626586293464e-07 0.08910782959671737 -4.75868046662109e-07" rpy="0 0 0"/>
     <mass value="11.601933377005569"/>
     <inertia ixx="0.066678" iyy="0.074767" izz="0.066678" ixy="-0.0" iyz="0.0" ixz="0.0"/>
   </inertial>
   <visual>
-    <origin xyz="-0.765818 0.289197 0.271208" rpy="0 0 0"/>
+    <origin xyz="-0.384314 0.452481 0.077336" rpy="0 0 0"/>
     <geometry>
       <mesh filename="package://robot_description/meshes/wheel_6.stl" scale="0.001 0.001 0.001"/>
@@ -218,5 +218,5 @@
   </visual>
   <collision>
-    <origin xyz="-0.765818 0.289197 0.271208" rpy="0 0 0"/>
+    <origin xyz="-0.384314 0.452481 0.077336" rpy="0 0 0"/>
     <geometry>
       <mesh filename="package://robot_description/meshes/wheel_6.stl" scale="0.001 0.001 0.001"/>
@@ -225,5 +225,5 @@
 </link>
 <joint name="Revolute 1" type="continuous">
-  <origin xyz="0.032254 -0.238359 0.327323" rpy="0 0 0"/>
+  <origin xyz="0.032254 -0.238359 0.15875" rpy="0 0 0"/>
   <parent link="base_link"/>
   <child link="right_big_pivot_1"/>
@@ -231,5 +231,5 @@
 </joint>
 <joint name="Revolute 3" type="continuous">
-  <origin xyz="0.032254 0.2386 0.327323" rpy="0 0 0"/>
+  <origin xyz="0.032254 0.2386 0.15875" rpy="0 0 0"/>
   <parent link="base_link"/>
   <child link="left_big_pivot_1"/>
@@ -255,5 +255,5 @@
 </joint>
 <joint name="Revolute 7" type="continuous">
-  <origin xyz="0.203219 -0.049812 0.465295" rpy="0 0 0"/>
+  <origin xyz="-0.178284 0.0 -0.07506" rpy="0 0 0"/>
   <parent link="right_little_pivot_1"/>
   <child link="wheel_2"/>
@@ -261,5 +261,5 @@
 </joint>
 <joint name="Revolute 8" type="continuous">
-  <origin xyz="0.558812 -0.047536 0.465295" rpy="0 0 0"/>
+  <origin xyz="0.177308 0.0 -0.077336" rpy="0 0 0"/>
   <parent link="right_little_pivot_1"/>
   <child link="wheel_3"/>
@@ -267,5 +267,5 @@
 </joint>
 <joint name="Revolute 9" type="continuous">
-  <origin xyz="0.00963 -0.211277 -0.18991" rpy="0 0 0"/>
+  <origin xyz="-0.349504 -0.003175 -0.254" rpy="0 0 0"/>
   <parent link="right_big_pivot_1"/>
   <child link="wheel_4"/>
@@ -273,5 +273,5 @@
 </joint>
 <joint name="Revolute 10" type="continuous">
-  <origin xyz="0.203219 0.161008 -0.439781" rpy="0 0 0"/>
+  <origin xyz="-0.178284 0.0 -0.07506" rpy="0 0 0"/>
   <parent link="left_little_pivot_1"/>
   <child link="wheel_5"/>
@@ -279,5 +279,5 @@
 </joint>
 <joint name="Revolute 11" type="continuous">
-  <origin xyz="0.558812 0.163284 -0.439781" rpy="0 0 0"/>
+  <origin xyz="0.177308 0.0 -0.077336" rpy="0 0 0"/>
   <parent link="left_little_pivot_1"/>
   <child link="wheel_6"/>

Commit message: try fix for xacro

File: robot_description/urdf/robot.xacro (robot description, xacro)
@@ -256,5 +256,5 @@
 <joint name="Revolute 7" type="continuous">
   <origin xyz="-0.178284 0.0 -0.07506" rpy="0 0 0"/>
-  <parent link="right_little_pivot_1"/>
+  <parent link="left_little_pivot_1"/>
   <child link="wheel_2"/>
   <axis xyz="-0.0 -1.0 -0.0"/>
@@ -262,5 +262,5 @@
 <joint name="Revolute 8" type="continuous">
   <origin xyz="0.177308 0.0 -0.077336" rpy="0 0 0"/>
-  <parent link="right_little_pivot_1"/>
+  <parent link="left_little_pivot_1"/>
   <child link="wheel_3"/>
   <axis xyz="0.0 1.0 0.0"/>
@@ -274,5 +274,5 @@
 <joint name="Revolute 10" type="continuous">
   <origin xyz="-0.178284 0.0 -0.07506" rpy="0 0 0"/>
-  <parent link="left_little_pivot_1"/>
+  <parent link="right_little_pivot_1"/>
   <child link="wheel_5"/>
   <axis xyz="-0.0 -1.0 -0.0"/>
@@ -280,5 +280,5 @@
 <joint name="Revolute 11" type="continuous">
   <origin xyz="0.177308 0.0 -0.077336" rpy="0 0 0"/>
-  <parent link="left_little_pivot_1"/>
+  <parent link="right_little_pivot_1"/>
   <child link="wheel_6"/>
   <axis xyz="0.0 1.0 0.0"/>

Commit message: replace again

File: robot_description/urdf/robot.xacro (robot description, xacro)
@@ -256,5 +256,5 @@
 <joint name="Revolute 7" type="continuous">
   <origin xyz="-0.178284 0.0 -0.07506" rpy="0 0 0"/>
-  <parent link="left_little_pivot_1"/>
+  <parent link="right_little_pivot_1"/>
   <child link="wheel_2"/>
   <axis xyz="-0.0 -1.0 -0.0"/>
@@ -262,5 +262,5 @@
 <joint name="Revolute 8" type="continuous">
   <origin xyz="0.177308 0.0 -0.077336" rpy="0 0 0"/>
-  <parent link="left_little_pivot_1"/>
+  <parent link="right_little_pivot_1"/>
   <child link="wheel_3"/>
   <axis xyz="0.0 1.0 0.0"/>
@@ -274,5 +274,5 @@
 <joint name="Revolute 10" type="continuous">
   <origin xyz="-0.178284 0.0 -0.07506" rpy="0 0 0"/>
-  <parent link="right_little_pivot_1"/>
+  <parent link="left_little_pivot_1"/>
   <child link="wheel_5"/>
   <axis xyz="-0.0 -1.0 -0.0"/>
@@ -280,5 +280,5 @@
 <joint name="Revolute 11" type="continuous">
   <origin xyz="0.177308 0.0 -0.077336" rpy="0 0 0"/>
-  <parent link="right_little_pivot_1"/>
+  <parent link="left_little_pivot_1"/>
   <child link="wheel_6"/>
   <axis xyz="0.0 1.0 0.0"/>
